File: RBG Light Controller/MainBoard.brd (EAGLE design)
At the start: 51.7 x 53.3 mm, 22 parts, among them IC1 74HC595N, IC2 4584N, U1 ARDUINOR3-BPLACE

Commit message: updated schematic
Routing:
- net N$24: track 75.5 -> 38.0 mm
- net N$23: track 63.1 -> 37.7 mm, vias 4 -> 1
- net RED: track 76.2 -> 52.4 mm, vias 1 -> 2
- net N$14: track 42.6 -> 25.4 mm, vias 1 -> 0
- net SWITCH2: track 90.1 -> 77.5 mm, vias 0 -> 2
- net N$6: track 61.7 -> 49.4 mm
- net N$2: track 32.1 -> 22.9 mm
- net SWITCH1: track 93.5 -> 85.9 mm, vias 1 -> 0
- net BLUE: track 51.8 -> 44.9 mm, vias 3 -> 1
- net GREEN: track 78.6 -> 72.2 mm, vias 2 -> 1
- net 12V: track 57.2 -> 51.3 mm, vias 4 -> 0
- net 5V: track 89.2 -> 84.7 mm, vias 1 -> 0
- net N$1: track 36.1 -> 32.1 mm
- net N$25: track 61.6 -> 57.7 mm, vias 1 -> 0
- net N$27: track 24.0 -> 20.7 mm
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